File: nodePWR.sch (KiCad schematic (older format))
At the start: 0 parts

Commit message: Checkpoint - starting PCB
On branch master
modified:   nodePWR-cache.lib
modified:   nodePWR.kicad_pcb
modified:   nodePWR.pro
modified:   nodePWR.sch
Parts:
- added BT1: LiFeP04, rockingdlabs:JST_PH_S2B-PH-SM4-TB_02x2.00mm_Angled, symbol Battery_Cell
- added C1: 1 uF, Capacitors_SMD:C_0603, symbol C
- added C2: 2 uF, Capacitors_SMD:C_0603, symbol C
- added D1: Charging, LEDs:LED_0603, symbol LED_Small
- added P1: Vin (4.5-30VDC), Pin_Headers:Pin_Header_Straight_1x02, symbol CONN_01X02
- added P2: USB (power only), Connect:USB_Micro-B_10103594-0001LF, symbol CONN_01X05
- added P3: Node, rockingdlabs:FPC_conn-6_8x4.9mm_Pitch0.5mm, symbol CONN_01X06
- added P4: Serial I/O, Pin_Headers:Pin_Header_Angled_1x06, symbol CONN_01X06
- added R1: 10k, Resistors_SMD:R_0603, symbol R
- added R2: 1k, Resistors_SMD:R_0603, symbol R
- added R3: 75, Resistors_SMD:R_0603, symbol R
- added R4: 490k, Resistors_SMD:R_0603, symbol R
- added R5: 100k, Resistors_SMD:R_0603, symbol R
- added SW1: Prgm, Buttons_Switches_SMD:SW_SPDT_PCM12, symbol SW_SPDT
- added U1: bq25070, Housings_DFN_QFN:DFN-10-1EP_2x3mm_Pitch0.5mm, symbol bq25070
Connections:
- new net: R2.1, U1.2 (IMON)
- new net: R4.2, R5.1, U1.5 (TS)
- new net: R1.1, U1.7 (CTRL)
- new net: D1.1 (K), U1.8 (CHG)
- new net: D1.2 (A), R3.2
- new net +3V3: R3.1, R4.1, U1.4 (LDO)
- new net +BATT: BT1.1 (+), C2.1, P3.6 (P6), U1.10 (OUT), U1.6 (BAT)
- new net GND: BT1.2 (-), C1.2, C2.2, P1.2 (P2), P2.5 (P5), P3.5 (P5), P4.6 (P6), R1.2, R2.2, R5.2, SW1.3 (C), U1.11 (PAD), U1.3 (GND), U1.9 (GND)
- new net PGM: P3.4 (P4), SW1.2 (B)
- new net RXD: P3.2 (P2), P4.3 (P3)
- new net TXD: P3.1 (P1), P4.2 (P2)
- new net VCC: P3.3 (P3), P4.4 (P4)
- new net VDD: C1.1, P1.1 (P1), P2.1 (P1), U1.1 (IN)
- no-connect marks 0 -> 6

Commit message: Use TI/Ultra-librarian footprint for bq25070
On branch master
modified:   nodePWR.kicad_pcb
modified:   nodePWR.sch
Parts:
- U1: footprint Housings_DFN_QFN:DFN-10-1EP_2x3mm_Pitch0.5mm -> rockingdlabs:bq25070_DQC_10-DQC10_P84X2P4
Changed lines of the file:
@@
 F 0 "U1" H 5050 4506 50  0000 C CNN
 F 1 "bq25070" H 5050 4415 50  0000 C CNN
-F 2 "Housings_DFN_QFN:DFN-10-1EP_2x3mm_Pitch0.5mm" H 5050 3850 50  0001 C CNN
+F 2 "rockingdlabs:bq25070_DQC_10-DQC10_P84X2P4" H 5050 3850 50  0001 C CNN
 F 3 "LiFePO4 Charger" H 5050 4324 50  0000 C CNN
 	1    5050 3850

Commit message: Make changes to allow for an enclosure
    - move USB closer to PCB edge
    - Rotate BT1 so that connector can be used when there is an
      enclosure.
    - Add pins to solder in a battery.
    - change serial I/O header to veritical.
Parts:
- added P5: BAT, Pin_Headers:Pin_Header_Straight_1x02, symbol CONN_01X02
- P4: footprint Pin_Headers:Pin_Header_Angled_1x06 -> Pin_Headers:Pin_Header_Straight_1x06
Connections:
- net +BATT: now also P5.1 (P1)
- net GND: now also P5.2 (P2)
Changed lines of the file:
@@
 F 0 "P4" H 5378 6891 50  0000 L CNN
 F 1 "Serial I/O" H 5378 6800 50  0000 L CNN
-F 2 "Pin_Headers:Pin_Header_Angled_1x06" H 5300 6850 50  0001 C CNN
+F 2 "Pin_Headers:Pin_Header_Straight_1x06" H 5300 6850 50  0001 C CNN
 F 3 "" H 5300 6850 50  0000 C CNN
 	1    5300 6850
@@
 $EndComp
 Wire Wire Line
-	4950 4550 4950 4600
+	4950 4600 4950 4550
 Wire Wire Line
 	3150 4600 5150 4600
@@
 	6050 3650 6050 3200
 Wire Wire Line
-	5950 3750 8150 3750
+	5950 3750 8750 3750
 Wire Wire Line
 	6050 3750 6050 4100
@@
 L +BATT #PWR014
 U 1 1 584F72A7
-P 8150 3750
-F 0 "#PWR014" H 8150 3600 50  0001 C CNN
-F 1 "+BATT" V 8165 3878 50  0000 L CNN
-F 2 "" H 8150 3750 50  0000 C CNN
-F 3 "" H 8150 3750 50  0000 C CNN
-	1    8150 3750
+P 8750 3750
+F 0 "#PWR014" H 8750 3600 50  0001 C CNN
+F 1 "+BATT" V 8765 3878 50  0000 L CNN
+F 2 "" H 8750 3750 50  0000 C CNN
+F 3 "" H 8750 3750 50  0000 C CNN
+	1    8750 3750
 	0    1    1    0
 $EndComp
 Connection ~ 7900 3750
+$Comp
+L CONN_01X02 P5
+U 1 1 5850A0EA
+P 8650 4100
+F 0 "P5" H 8728 4141 50  0000 L CNN
+F 1 "BAT" H 8728 4050 50  0000 L CNN
+F 2 "Pin_Headers:Pin_Header_Straight_1x02" H 8650 4100 50  0001 C CNN
+F 3 "" H 8650 4100 50  0000 C CNN
+	1    8650 4100
+	1    0    0    -1
+$EndComp
+Wire Wire Line
+	8450 4050 8350 4050
+Wire Wire Line
+	8350 4050 8350 3750
+Connection ~ 8350 3750
+Wire Wire Line
+	7900 4250 8450 4250
+Wire Wire Line
+	8450 4250 8450 4150
+Connection ~ 7900 4250
 $EndSCHEMATC

Commit message: Change to standard resistor value
On branch master
modified:   nodePWR.sch
Parts:
- R4: value 490k -> 487k
Changed lines of the file:
@@
 P 7100 2750
 F 0 "R4" H 7170 2796 50  0000 L CNN
-F 1 "490k" H 7170 2705 50  0000 L CNN
+F 1 "487k" H 7170 2705 50  0000 L CNN
 F 2 "Resistors_SMD:R_0603" V 7030 2750 50  0001 C CNN
 F 3 "" H 7100 2750 50  0000 C CNN

Commit message: Checkpoint - replaced 6pin conn with 7pin
    - Changed signals to provide charge controll and monitoring on P3
Parts:
- removed D1: Charging, LEDs:LED_0603, symbol LED_Small
- removed P3: Node, rockingdlabs:FPC_conn-6_8x4.9mm_Pitch0.5mm, symbol CONN_01X06
- removed R3: 75, Resistors_SMD:R_0603, symbol R
- added P3: Node, symbol CONN_01X07
Connections:
- net labels added: CHRG, CTRL
- net labels removed: VCC
- wire segments 56 -> 68
- no-connect marks 6 -> 7
Changed lines of the file:
@@
 $EndDescr
-$Comp
-L CONN_01X06 P3
-U 1 1 584F4021
-P 2200 6950
-F 0 "P3" H 2278 6991 50  0000 L CNN
-F 1 "Node" H 2278 6900 50  0000 L CNN
-F 2 "rockingdlabs:FPC_conn-6_8x4.9mm_Pitch0.5mm" H 2200 6950 50  0001 C CNN
-F 3 "" H 2200 6950 50  0000 C CNN
-	1    2200 6950
-	-1   0    0    -1
-$EndComp
 $Comp
 L CONN_01X05 P2
@@
 	1700 1100 2100 1100
 Wire Wire Line
-	2100 950  2100 1700
+	2100 950  2100 1100
+Wire Wire Line
+	2100 1100 2100 1700
 Wire Wire Line
 	2100 1700 1700 1700
@@
 $EndComp
 $Comp
-L LED_Small D1
-U 1 1 584F4F64
-P 6050 3100
-F 0 "D1" V 6096 3032 50  0000 R CNN
-F 1 "Charging" V 6005 3032 50  0000 R CNN
-F 2 "LEDs:LED_0603" V 6050 3100 50  0001 C CNN
-F 3 "" V 6050 3100 50  0000 C CNN
-	1    6050 3100
-	0    -1   -1   0
-$EndComp
-$Comp
-L R R3
-U 1 1 584F5004
-P 6050 2750
-F 0 "R3" H 6120 2796 50  0000 L CNN
-F 1 "75" H 6120 2705 50  0000 L CNN
-F 2 "Resistors_SMD:R_0603" V 5980 2750 50  0001 C CNN
-F 3 "" H 6050 2750 50  0000 C CNN
-	1    6050 2750
-	1    0    0    -1
-$EndComp
-$Comp
 L GND #PWR04
 U 1 1 584F556F
@@
 	2400 6800 5100 6800
 Wire Wire Line
-	2400 7000 3850 7000
-Wire Wire Line
-	3850 7000 3850 6050
+	2400 6900 3850 6900
+Wire Wire Line
+	3850 6900 3850 6050
 Wire Wire Line
 	3850 6050 4000 6050
@@
 $EndComp
 Wire Wire Line
-	2400 6900 5100 6900
-Wire Wire Line
-	2400 7100 5100 7100
-Wire Wire Line
-	2650 7100 2650 7400
-Wire Wire Line
-	2400 7200 3150 7200
-Connection ~ 2650 7100
+	2400 7200 2650 7200
+Wire Wire Line
+	2650 7200 5100 7200
+Wire Wire Line
+	2650 7200 2650 7400
+Wire Wire Line
+	2400 7300 3150 7300
+Connection ~ 2650 7200
 NoConn ~ 5100 7000
 $Comp
@@
 $EndComp
 Wire Wire Line
-	3150 7200 3150 6300
+	3150 7300 3150 6300
 $Comp
 L CONN_01X06 P4
@@
 RXD
 Text Label 2550 6900 0    60   ~ 0
-VCC
-Text Label 2550 7000 0    60   ~ 0
 PGM
 NoConn ~ 5100 6600
@@
 L +3V3 #PWR07
 U 1 1 584F5E3F
-P 6350 2400
-F 0 "#PWR07" H 6350 2250 50  0001 C CNN
-F 1 "+3V3" H 6365 2573 50  0000 C CNN
-F 2 "" H 6350 2400 50  0000 C CNN
-F 3 "" H 6350 2400 50  0000 C CNN
-	1    6350 2400
+P 7100 2450
+F 0 "#PWR07" H 7100 2300 50  0001 C CNN
+F 1 "+3V3" H 7115 2623 50  0000 C CNN
+F 2 "" H 7100 2450 50  0000 C CNN
+F 3 "" H 7100 2450 50  0000 C CNN
+	1    7100 2450
 	1    0    0    -1
 $EndComp
@@
 	4950 4600 4950 4550
 Wire Wire Line
-	3150 4600 5150 4600
+	3150 4600 3600 4600
+Wire Wire Line
+	3600 4600 4000 4600
+Wire Wire Line
+	4000 4600 4950 4600
+Wire Wire Line
+	4950 4600 5050 4600
+Wire Wire Line
+	5050 4600 5150 4600
 Wire Wire Line
 	5150 4600 5150 4550
 Wire Wire Line
-	5050 4550 5050 4650
+	5050 4550 5050 4600
+Wire Wire Line
+	5050 4600 5050 4650
 Connection ~ 5050 4600
-Wire Wire Line
-	6050 2450 7100 2450
-Wire Wire Line
-	6050 2450 6050 2600
-Wire Wire Line
-	6050 2900 6050 3000
-Wire Wire Line
-	6350 2400 6350 2450
-Connection ~ 6350 2450
 $Comp
 L C C2
@@
 	5950 3650 6050 3650
 Wire Wire Line
-	6050 3650 6050 3200
-Wire Wire Line
-	5950 3750 8750 3750
-Wire Wire Line
-	6050 3750 6050 4100
+	5950 3750 6050 3750
+Wire Wire Line
+	6050 3750 7900 3750
+Wire Wire Line
+	7900 3750 8350 3750
+Wire Wire Line
+	8350 3750 8750 3750
+Wire Wire Line
+	6050 3750 6050 3850
+Wire Wire Line
+	6050 3850 6050 4100
 Wire Wire Line
 	5950 3850 6050 3850
@@
 $EndComp
 Wire Wire Line
-	7900 4200 7900 4350
+	7900 4200 7900 4250
+Wire Wire Line
+	7900 4250 7900 4350
 Wire Wire Line
 	6050 4400 6050 4550
@@
 	7100 2450 7100 2600
 Wire Wire Line
-	7100 2900 7100 3100
+	7100 2900 7100 3000
+Wire Wire Line
+	7100 3000 7100 3100
 Wire Wire Line
 	7100 3400 7100 3500
@@
 $EndComp
 Wire Wire Line
-	2850 3650 4150 3650
+	2850 3650 3150 3650
+Wire Wire Line
+	3150 3650 4150 3650
 $Comp
 L R R1
@@
 	4000 3850 4000 4050
 Wire Wire Line
-	4150 3750 3600 3750
+	3350 3750 3600 3750
+Wire Wire Line
+	3600 3750 4150 3750
 Wire Wire Line
 	3600 3750 3600 4050
@@
 	8450 4250 8450 4150
 Connection ~ 7900 4250
+$Comp
+L CONN_01X07 P3
+U 1 1 58641C15
+P 2200 7000
+F 0 "P3" H 2278 7041 50  0000 L CNN
+F 1 "Node" H 2278 6950 50  0000 L CNN
+F 2 "" H 2200 7000 50  0000 C CNN
+F 3 "" H 2200 7000 50  0000 C CNN
+	1    2200 7000
+	-1   0    0    -1
+$EndComp
+Wire Wire Line
+	5100 7200 5100 7100
+NoConn ~ 5100 6900
+Wire Wire Line
+	2400 7000 2900 7000
+Wire Wire Line
+	2400 7100 2900 7100
+Text Label 2550 7000 0    60   ~ 0
+CTRL
+Text Label 2550 7100 0    60   ~ 0
+CHRG
+Connection ~ 3600 3750
+Text Label 3350 3750 0    60   ~ 0
+CTRL
+Text Label 6000 3650 0    60   ~ 0
+CHRG
 $EndSCHEMATC

Commit message: Checkpoint - Re-annotate, fix DRC warnings
    - Renumbered all anotations to eliminate gaps
    - Marked VDD and GND as power

On branch addChargerSignals
modified:   nodePWR-cache.lib
modified:   nodePWR.sch
Parts:
- renumbered R4 to R3, R5 to R4
Connections:
- wire segments 68 -> 53
Changed lines of the file:
@@
 $EndComp
 Wire Wire Line
-	1700 2100 1850 2100
+	1700 2100 2250 2100
 Wire Wire Line
 	1850 2100 1850 2150
@@
 $EndComp
 Wire Wire Line
-	1700 1100 2100 1100
-Wire Wire Line
-	2100 950  2100 1100
-Wire Wire Line
-	2100 1100 2100 1700
+	1700 1100 2300 1100
+Wire Wire Line
+	2100 950  2100 1700
 Wire Wire Line
 	2100 1700 1700 1700
@@
 $EndComp
 Wire Wire Line
-	2400 7200 2650 7200
-Wire Wire Line
-	2650 7200 5100 7200
+	2400 7200 5100 7200
 Wire Wire Line
 	2650 7200 2650 7400
@@
 	4950 4600 4950 4550
 Wire Wire Line
-	3150 4600 3600 4600
-Wire Wire Line
-	3600 4600 4000 4600
-Wire Wire Line
-	4000 4600 4950 4600
-Wire Wire Line
-	4950 4600 5050 4600
-Wire Wire Line
-	5050 4600 5150 4600
+	3150 4600 5150 4600
 Wire Wire Line
 	5150 4600 5150 4550
 Wire Wire Line
-	5050 4550 5050 4600
-Wire Wire Line
-	5050 4600 5050 4650
+	5050 4550 5050 4650
 Connection ~ 5050 4600
 $Comp
@@
 	5950 3650 6050 3650
 Wire Wire Line
-	5950 3750 6050 3750
-Wire Wire Line
-	6050 3750 7900 3750
-Wire Wire Line
-	7900 3750 8350 3750
-Wire Wire Line
-	8350 3750 8750 3750
-Wire Wire Line
-	6050 3750 6050 3850
-Wire Wire Line
-	6050 3850 6050 4100
+	5950 3750 8750 3750
+Wire Wire Line
+	6050 3750 6050 4100
 Wire Wire Line
 	5950 3850 6050 3850
@@
 $EndComp
 Wire Wire Line
-	7900 4200 7900 4250
-Wire Wire Line
-	7900 4250 7900 4350
+	7900 4200 7900 4350
 Wire Wire Line
 	6050 4400 6050 4550
 $Comp
-L R R4
+L R R3
 U 1 1 584F66B5
 P 7100 2750
-F 0 "R4" H 7170 2796 50  0000 L CNN
+F 0 "R3" H 7170 2796 50  0000 L CNN
 F 1 "487k" H 7170 2705 50  0000 L CNN
 F 2 "Resistors_SMD:R_0603" V 7030 2750 50  0001 C CNN
@@
 $EndComp
 $Comp
-L R R5
+L R R4
 U 1 1 584F6737
 P 7100 3250
-F 0 "R5" H 7170 3296 50  0000 L CNN
+F 0 "R4" H 7170 3296 50  0000 L CNN
 F 1 "100k" H 7170 3205 50  0000 L CNN
 F 2 "Resistors_SMD:R_0603" V 7030 3250 50  0001 C CNN
@@
 	7100 2450 7100 2600
 Wire Wire Line
-	7100 2900 7100 3000
-Wire Wire Line
-	7100 3000 7100 3100
+	7100 2900 7100 3100
 Wire Wire Line
 	7100 3400 7100 3500
@@
 $EndComp
 Wire Wire Line
-	2850 3650 3150 3650
-Wire Wire Line
-	3150 3650 4150 3650
+	2850 3650 4150 3650
 $Comp
 L R R1
@@
 	4000 3850 4000 4050
 Wire Wire Line
-	3350 3750 3600 3750
-Wire Wire Line
-	3600 3750 4150 3750
+	3350 3750 4150 3750
 Wire Wire Line
 	3600 3750 3600 4050
@@
 Text Label 6000 3650 0    60   ~ 0
 CHRG
+$Comp
+L PWR_FLAG #FLG015
+U 1 1 58642A49
+P 2300 1100
+F 0 "#FLG015" H 2300 1175 50  0001 C CNN
+F 1 "PWR_FLAG" H 2300 1274 50  0000 C CNN
+F 2 "" H 2300 1100 50  0000 C CNN
+F 3 "" H 2300 1100 50  0000 C CNN
+	1    2300 1100
+	1    0    0    -1
+$EndComp
+$Comp
+L PWR_FLAG #FLG016
+U 1 1 58642B12
+P 2250 2100
+F 0 "#FLG016" H 2250 2175 50  0001 C CNN
+F 1 "PWR_FLAG" H 2250 2274 50  0000 C CNN
+F 2 "" H 2250 2100 50  0000 C CNN
+F 3 "" H 2250 2100 50  0000 C CNN
+	1    2250 2100
+	1    0    0    -1
+$EndComp
+Connection ~ 1850 2100
 $EndSCHEMATC

Commit message: Add footprint for 7pin
On branch addChargerSignals
modified:   nodePWR.net
modified:   nodePWR.sch
Parts:
- P3: footprint (none) -> rockingdlabs:FPC_conn-7_8x4.9mm_Pitch0.5mm
Changed lines of the file:
@@
 F 0 "P3" H 2278 7041 50  0000 L CNN
 F 1 "Node" H 2278 6950 50  0000 L CNN
-F 2 "" H 2200 7000 50  0000 C CNN
+F 2 "rockingdlabs:FPC_conn-7_8x4.9mm_Pitch0.5mm" H 2200 7000 50  0001 C CNN
 F 3 "" H 2200 7000 50  0000 C CNN
 	1    2200 7000
